Commit message: Start to check if TFs are good

File: catkin_ws/src/sensor-tools/urdf/sensor-box.urdf (robot description, URDF)
Before this commit: robot sensor_box, 9 links, 8 joints
Joints:
- joint mynt_bottom_link_to_mynt_link: origin xyz=0.0628 0.0105 0.01573 rpy=0.0 0.0 0.0 -> xyz=-0.0628 0.0105 0.01573 rpy=0 0 1.2

Commit message: Adjust TF, prepare to record first session

File: catkin_ws/src/sensor-tools/urdf/sensor-box.urdf (robot description, URDF)
Before this commit: robot sensor_box, 9 links, 8 joints
Joints:
- joint mynt_bottom_link_to_mynt_link: origin xyz=-0.0628 0.0105 0.0136 rpy=0 0 1.2 -> xyz=0.0 0.01 0.0136 rpy=0 0 0.91

Commit message: Adjust Mynt TF

File: catkin_ws/src/sensor-tools/urdf/sensor-box.urdf (robot description, URDF)
Before this commit: robot sensor_box, 9 links, 8 joints
Joints:
- joint mynt_bottom_link_to_mynt_link: origin xyz=0.0 0.01 0.0136 rpy=0 0 0.91 -> xyz=0.0 0.01 0.0136 rpy=0 0 0.78

Commit message: steam deck with podman

File: catkin_ws/src/sensor-tools/urdf/sensor-box.urdf (robot description, URDF)
Before this commit: robot sensor_box, 9 links, 8 joints
Links:
- added link aft_mapped
Joints:
- added joint aft_mapped_to_base_link: type fixed, parent aft_mapped, child base_link, origin xyz=-0.0404 0 -0.264 rpy=0 0 0

Commit message: Velarray integrated. Rafaela Thesis

File: catkin_ws/src/sensor-tools/urdf/sensor-box.urdf (robot description, URDF)
Before this commit: robot sensor_box, 10 links, 9 joints
Links:
- removed link aft_mapped
- removed link base_sensor_box
- removed link livox_frame
- removed link mynteye_bottom_screw_frame
- removed link mynteye_link
- removed link realsense_bottom_screw_frame
- removed link xsens_base
- removed link xsens_frame
- added link antenna_link
- added link base_apparatus
- added link mynt_bottom_screw_link
- added link mynt_link
- added link velarray_link
- added link xsens_link
- link base_link: geometry visual mesh filename=package://urdf_tutorial/my_meshes/apparatus_box.stl scale=1 1 1
Joints:
- removed joint aft_mapped_to_base_link
- removed joint base_link_to_base_sensor_box
- removed joint base_sensor_box_to_livox
- removed joint base_sensor_box_to_mynt_bottom_screw
- removed joint base_sensor_box_to_realsense
- removed joint base_sensor_box_to_xsens
- removed joint mynt_bottom_link_to_mynt_link
- removed joint realsense_bottom_screw_to_realsense
- removed joint xsens_to_original_xsense
- added joint base to_bottom_mynt_screw: type fixed, parent base_apparatus, child mynt_bottom_screw_link, origin xyz=-0.031088 0.014078 0.146 rpy=0 0 0.802851456
- added joint base_link_to_base_apparatus: type fixed, parent base_link, child base_apparatus, origin xyz=0 0 0 rpy=0 0 -1.570796327
- added joint base_to_antenna: type fixed, parent base_apparatus, child antenna_link, origin xyz=-0.002106 -0.036673 0.3549896 rpy=0 0 0
- added joint base_to_realsense: type fixed, parent base_apparatus, child realsense_link, origin xyz=-0.045984 0.065623 0.0415 rpy=-1.570796327 0 0
- added joint base_to_velarray: type fixed, parent base_apparatus, child velarray_link, origin xyz=0.041541 0.072093 0.269396 rpy=0 0 0
- added joint base_to_xsens: type fixed, parent base_apparatus, child xsens_link, origin xyz=-0.017534 -0.029827 0.015160 rpy=0 0 0
- added joint mynt_screw_to_mynt_frame: type fixed, parent mynt_bottom_screw_link, child mynt_link, origin xyz=-0.059939 0.005 0.014600 rpy=0 0 0
