Commit message: Add ROS package dependencies as git submodules
- realsense-ros: RealSense camera driver
- norlab_xsens_driver: Xsens IMU driver (jazzy branch)
- ouster-ros: Ouster LiDAR driver (ros2 branch)
- hector_recorder: Recording and mapping tools
- nmea_navsat_driver: NMEA navigation driver (ros2 branch)

Submodules enable:
- Easier dependency management
- Clean separation between app and dependencies
- Version pinning per commit
- Recursive cloning of all sources

File: docker_ws/src/apparatus_description/urdf/robot.urdf.xacro (robot description, xacro)
@@ -1,5 +1,5 @@
 <?xml version="1.0"?>
 <robot xmlns:xacro="http://www.ros.org/wiki/xacro" name="robot">
-<xacro:property name="mesh_dir" value="/home/tobias/Development/fruc_dataset_apparatus/docker/docker_shared/apparatus_description/meshes"/>
+<xacro:property name="mesh_dir" value="$(find apparatus_description)/meshes"/>
 <!-- Mesh path prefix -->
 <xacro:property name="mesh_prefix" value="package://apparatus_description/meshes" />
